File: hardware/led controller/led controller/led controller.kicad_sch (KiCad schematic)
At the start: 4 parts, among them J1 Conn_01x03, J2 Conn_01x03, J3 Conn_01x02

Commit message: Update PCB
Parts:
- added J4, J5: Conn_01x15_Male, symbol Connector:Conn_01x15_Male
Connections:
- net +5V: now also J5.1 (Pin_1)
- net GND: now also J4.4 (Pin_4), J5.2 (Pin_2)
- net I2C_SCL: now also J5.7 (Pin_7)
- net I2C_SDA: now also J5.8 (Pin_8)
- net LED_D_OUT: now also J4.5 (Pin_5)
- net D1: now reaches A1.1 (D1/TX)
- net D1: now also J4.1 (Pin_1)
- net D7: now reaches A1.10 (D7)
- net D7: now also J4.10 (Pin_10)
- net D8: now reaches A1.11 (D8)
- net D8: now also J4.11 (Pin_11)
- net D9: now reaches A1.12 (D9)
- net D9: now also J4.12 (Pin_12)
- net D10: now reaches A1.13 (D10)
- net D10: now also J4.13 (Pin_13)
- net D11: now reaches A1.14 (D11)
- net D11: now also J4.14 (Pin_14)
- net D12: now reaches A1.15 (D12)
- net D12: now also J4.15 (Pin_15)
- net D13: now reaches A1.16 (D13)
- net D13: now also J5.15 (Pin_15)
- net +3.3V: now reaches A1.17 (3V3)
- net +3.3V: now also J5.14 (Pin_14)
- net AREF: now reaches A1.18 (AREF)
- net AREF: now also J5.13 (Pin_13)
- net A0: now reaches A1.19 (A0)
- net A0: now also J5.12 (Pin_12)
- net D0: now reaches A1.2 (D0/RX)
- net D0: now also J4.2 (Pin_2)
- net A1: now reaches A1.20 (A1)
- net A1: now also J5.11 (Pin_11)
- net A2: now reaches A1.21 (A2)
- net A2: now also J5.10 (Pin_10)
- net A3: now reaches A1.22 (A3)
- net A3: now also J5.9 (Pin_9)
- net A6: now reaches A1.25 (A6)
- net A6: now also J5.6 (Pin_6)
- net A7: now reaches A1.26 (A7)
- net A7: now also J5.5 (Pin_5)
- net VCC: now reaches A1.27 (+5V)
- net VCC: now also J5.4 (Pin_4)
- net RST: now reaches A1.28 (~{RESET})
- net RST: now also A1.3 (~{RESET}), J4.3 (Pin_3), J5.3 (Pin_3)
- net D3: now reaches A1.6 (D3)
- net D3: now also J4.6 (Pin_6)
- net D4: now reaches A1.7 (D4)
- net D4: now also J4.7 (Pin_7)
- net D5: now reaches A1.8 (D5)
- net D5: now also J4.8 (Pin_8)
- net D6: now reaches A1.9 (D6)
- net D6: now also J4.9 (Pin_9)
- no-connect marks 24 -> 0
